File: PC8801mkII VGA.sch (KiCad schematic (older format))
At the start: 5 parts

Commit message: Use the 3-row right angle VGA connector which is all digikey seems to have
Parts:
- V1: footprint Connector_Dsub:DSUB-15_Female_Horizontal_P2.77x2.84mm_EdgePinOffset4.94mm_Housed_MountingHolesOffset7.48mm -> Connector_Dsub:DSUB-15-HD_Female_Horizontal_P2.29x1.98mm_EdgePinOffset3.03mm_Housed_MountingHolesOffset4.94mm
Changed lines of the file:
@@
 F 0 "V1" H 7425 4367 50  0000 C CNN
 F 1 "15kHz VGA" H 7425 4276 50  0000 C CNN
-F 2 "Connector_Dsub:DSUB-15_Female_Horizontal_P2.77x2.84mm_EdgePinOffset4.94mm_Housed_MountingHolesOffset7.48mm" H 6475 3900 50  0001 C CNN
+F 2 "Connector_Dsub:DSUB-15-HD_Female_Horizontal_P2.29x1.98mm_EdgePinOffset3.03mm_Housed_MountingHolesOffset4.94mm" H 6475 3900 50  0001 C CNN
 F 3 " ~" H 6475 3900 50  0001 C CNN
 	1    7425 3500

Commit message: Revision with ACTUAL PARTS
Parts:
- N1: footprint Pin_Headers:Pin_Header_Straight_1x08_Pitch2.54mm -> SDS-80J:CUI_SDS-80J
- V1: footprint Connector_Dsub:DSUB-15-HD_Female_Horizontal_P2.29x1.98mm_EdgePinOffset3.03mm_Housed_MountingHolesOffset4.94mm -> Connector_TE_AMP_HD15:1-1734530-1
Connections:
- net labels added: Blue_VGA, Green_VGA, Red_VGA
Changed lines of the file:
@@
 F 0 "N1" H 5225 2222 50  0000 C CNN
 F 1 "PC88 RGB" H 5225 2313 50  0000 C CNN
-F 2 "Pin_Headers:Pin_Header_Straight_1x08_Pitch2.54mm" H 5225 2700 50  0001 C CNN
+F 2 "SDS-80J:CUI_SDS-80J" H 5225 2700 50  0001 C CNN
 F 3 "http://www.mouser.com/ds/2/18/40_c091_abd_e-75918.pdf" H 5225 2700 50  0001 C CNN
 	1    5225 2700
@@
 F 0 "V1" H 7425 4367 50  0000 C CNN
 F 1 "15kHz VGA" H 7425 4276 50  0000 C CNN
-F 2 "Connector_Dsub:DSUB-15-HD_Female_Horizontal_P2.29x1.98mm_EdgePinOffset3.03mm_Housed_MountingHolesOffset4.94mm" H 6475 3900 50  0001 C CNN
+F 2 "Connector_TE_AMP_HD15:1-1734530-1" H 6475 3900 50  0001 C CNN
 F 3 " ~" H 6475 3900 50  0001 C CNN
 	1    7425 3500
@@
 $EndComp
 Text Label 7125 3100 2    50   ~ 0
-Red
+Red_VGA
 Text Label 7125 3300 2    50   ~ 0
-Green
+Green_VGA
 Text Label 7125 3500 2    50   ~ 0
-Blue
+Blue_VGA
 Text Label 7125 3900 2    50   ~ 0
 GND

Commit message: Revised schematic based on the female pinout
Connections:
- net labels added: NC
- wire segments 30 -> 31
Changed lines of the file:
@@
 GND
 Text Label 4925 2600 2    50   ~ 0
+Green
+Text Label 5525 2600 0    50   ~ 0
 Red
-Text Label 5525 2600 0    50   ~ 0
-Green
 Text Label 5225 2400 0    50   ~ 0
 Blue
 Text Label 4925 2700 2    50   ~ 0
-12V
+NC
 NoConn ~ 5525 2700
 Text Label 4925 2800 2    50   ~ 0
+V-Sync
+Text Label 5525 2800 0    50   ~ 0
 H-Sync
-Text Label 5525 2800 0    50   ~ 0
-V-Sync
 $Comp
 L Connector:DB15_Female_HighDensity V1
@@
 	7125 3100 6850 3100
 Wire Wire Line
-	4325 3100 4325 2600
-Wire Wire Line
 	4325 2600 4925 2600
 Wire Wire Line
@@
 	6350 2400 6350 3500
 Wire Wire Line
-	6350 3500 6550 3500
-Wire Wire Line
 	5525 2600 6425 2600
-Wire Wire Line
-	6425 2600 6425 3300
-Wire Wire Line
-	6425 3300 6550 3300
 Wire Wire Line
 	5525 2800 8550 2800
 Wire Wire Line
-	8550 2800 8550 3700
-Wire Wire Line
-	8550 3700 7725 3700
-Wire Wire Line
 	4925 2800 4925 4175
-Wire Wire Line
-	4925 4175 8450 4175
-Wire Wire Line
-	8450 4175 8450 3500
-Wire Wire Line
-	8450 3500 7725 3500
 NoConn ~ 4925 2700
 $Comp
@@
 	0    1    1    0
 $EndComp
-Wire Wire Line
-	6550 3100 4325 3100
 $Comp
 L Device:R R2
@@
 Wire Wire Line
 	6850 3500 7125 3500
+Text Label 5525 2700 0    50   ~ 0
+12V
+Wire Wire Line
+	8550 2800 8550 3500
+Wire Wire Line
+	8550 3500 7725 3500
+Wire Wire Line
+	8550 4175 8550 3700
+Wire Wire Line
+	8550 3700 7725 3700
+Wire Wire Line
+	4925 4175 8550 4175
+Wire Wire Line
+	6350 3500 6550 3500
+Wire Wire Line
+	6425 2600 6425 3100
+Wire Wire Line
+	6425 3100 6550 3100
+Wire Wire Line
+	4325 2600 4325 3375
+Wire Wire Line
+	4325 3375 6550 3375
+Wire Wire Line
+	6550 3375 6550 3300
 $EndSCHEMATC

Commit message: Flipped version using fixed footprint
Parts:
- V1: footprint Connector_TE_AMP_HD15:1-1734530-1 -> Connector_TE_AMP_HD15:FIXED-1-1734530-1
Connections:
- net labels added: KEY
- wire segments 31 -> 35
- no-connect marks 6 -> 7
Changed lines of the file:
@@
 EESchema Schematic File Version 4
-LIBS:PC8801mkII VGA-cache
 EELAYER 26 0
 EELAYER END
@@
 Comment4 ""
 $EndDescr
-$Comp
-L Connector:DIN-8 N1
-U 1 1 5B82E0CE
-P 5225 2700
-F 0 "N1" H 5225 2222 50  0000 C CNN
-F 1 "PC88 RGB" H 5225 2313 50  0000 C CNN
-F 2 "SDS-80J:CUI_SDS-80J" H 5225 2700 50  0001 C CNN
-F 3 "http://www.mouser.com/ds/2/18/40_c091_abd_e-75918.pdf" H 5225 2700 50  0001 C CNN
-	1    5225 2700
-	-1   0    0    1
-$EndComp
 Text Label 5225 3000 0    50   ~ 0
 GND
 Text Label 4925 2600 2    50   ~ 0
+Red
+Text Label 5525 2600 0    50   ~ 0
 Green
-Text Label 5525 2600 0    50   ~ 0
-Red
 Text Label 5225 2400 0    50   ~ 0
 Blue
@@
 NoConn ~ 5525 2700
 Text Label 4925 2800 2    50   ~ 0
+H-Sync
+Text Label 5525 2800 0    50   ~ 0
 V-Sync
-Text Label 5525 2800 0    50   ~ 0
-H-Sync
 $Comp
 L Connector:DB15_Female_HighDensity V1
@@
 F 0 "V1" H 7425 4367 50  0000 C CNN
 F 1 "15kHz VGA" H 7425 4276 50  0000 C CNN
-F 2 "Connector_TE_AMP_HD15:1-1734530-1" H 6475 3900 50  0001 C CNN
+F 2 "Connector_TE_AMP_HD15:FIXED-1-1734530-1" H 6475 3900 50  0001 C CNN
 F 3 " ~" H 6475 3900 50  0001 C CNN
 	1    7425 3500
@@
 GND
 Text Label 7125 3600 2    50   ~ 0
-GND
+KEY
 Text Label 7125 3800 2    50   ~ 0
 GND
 NoConn ~ 7125 3700
 Text Label 7725 3500 0    50   ~ 0
+V-Sync
+Text Label 7725 3700 0    50   ~ 0
 H-Sync
-Text Label 7725 3700 0    50   ~ 0
-V-Sync
 NoConn ~ 7725 3900
 NoConn ~ 7725 3300
@@
 	5225 3800 5225 3900
 Wire Wire Line
-	7125 3600 5225 3600
-Connection ~ 5225 3600
-Wire Wire Line
-	5225 3600 5225 3800
-Wire Wire Line
 	7125 3400 5225 3400
 Connection ~ 5225 3400
-Wire Wire Line
-	5225 3400 5225 3600
 Wire Wire Line
 	7125 3200 5225 3200
@@
 Wire Wire Line
 	7125 3000 5225 3000
-Connection ~ 5225 3000
-Wire Wire Line
-	7125 3100 6850 3100
-Wire Wire Line
-	4325 2600 4925 2600
-Wire Wire Line
-	5225 2400 6350 2400
-Wire Wire Line
-	6350 2400 6350 3500
-Wire Wire Line
-	5525 2600 6425 2600
-Wire Wire Line
-	5525 2800 8550 2800
-Wire Wire Line
-	4925 2800 4925 4175
 NoConn ~ 4925 2700
 $Comp
 L Device:R R1
 U 1 1 5B82F80D
-P 6700 3100
-F 0 "R1" V 6493 3100 50  0000 C CNN
-F 1 "150" V 6584 3100 50  0000 C CNN
-F 2 "Resistors_ThroughHole:R_Axial_DIN0204_L3.6mm_D1.6mm_P5.08mm_Horizontal" V 6630 3100 50  0001 C CNN
-F 3 "~" H 6700 3100 50  0001 C CNN
-	1    6700 3100
+P 6175 4150
+F 0 "R1" V 5968 4150 50  0000 C CNN
+F 1 "150" V 6059 4150 50  0000 C CNN
+F 2 "Resistors_ThroughHole:R_Axial_DIN0204_L3.6mm_D1.6mm_P5.08mm_Horizontal" V 6105 4150 50  0001 C CNN
+F 3 "~" H 6175 4150 50  0001 C CNN
+	1    6175 4150
 	0    1    1    0
 $EndComp
@@
 L Device:R R2
 U 1 1 5B82FD72
-P 6700 3300
-F 0 "R2" V 6493 3300 50  0000 C CNN
-F 1 "150" V 6584 3300 50  0000 C CNN
-F 2 "Resistors_ThroughHole:R_Axial_DIN0204_L3.6mm_D1.6mm_P5.08mm_Horizontal" V 6630 3300 50  0001 C CNN
-F 3 "~" H 6700 3300 50  0001 C CNN
-	1    6700 3300
+P 6175 4475
+F 0 "R2" V 5968 4475 50  0000 C CNN
+F 1 "150" V 6059 4475 50  0000 C CNN
+F 2 "Resistors_ThroughHole:R_Axial_DIN0204_L3.6mm_D1.6mm_P5.08mm_Horizontal" V 6105 4475 50  0001 C CNN
+F 3 "~" H 6175 4475 50  0001 C CNN
+	1    6175 4475
 	0    1    1    0
 $EndComp
-Wire Wire Line
-	6850 3300 7125 3300
 $Comp
 L Device:R R3
 U 1 1 5B82FE62
-P 6700 3500
-F 0 "R3" V 6493 3500 50  0000 C CNN
-F 1 "150" V 6584 3500 50  0000 C CNN
-F 2 "Resistors_ThroughHole:R_Axial_DIN0204_L3.6mm_D1.6mm_P5.08mm_Horizontal" V 6630 3500 50  0001 C CNN
-F 3 "~" H 6700 3500 50  0001 C CNN
-	1    6700 3500
+P 6175 4750
+F 0 "R3" V 5968 4750 50  0000 C CNN
+F 1 "150" V 6059 4750 50  0000 C CNN
+F 2 "Resistors_ThroughHole:R_Axial_DIN0204_L3.6mm_D1.6mm_P5.08mm_Horizontal" V 6105 4750 50  0001 C CNN
+F 3 "~" H 6175 4750 50  0001 C CNN
+	1    6175 4750
 	0    1    1    0
 $EndComp
@@
 12V
 Wire Wire Line
-	8550 2800 8550 3500
+	5225 3400 5225 3800
+NoConn ~ 7125 3600
+Connection ~ 5225 3000
+$Comp
+L Connector:DIN-8 N1
+U 1 1 5B82E0CE
+P 5225 2700
+F 0 "N1" H 5225 2222 50  0000 C CNN
+F 1 "PC88 RGB" H 5225 2313 50  0000 C CNN
+F 2 "SDS-80J:CUI_SDS-80J" H 5225 2700 50  0001 C CNN
+F 3 "http://www.mouser.com/ds/2/18/40_c091_abd_e-75918.pdf" H 5225 2700 50  0001 C CNN
+	1    5225 2700
+	-1   0    0    1
+$EndComp
 Wire Wire Line
-	8550 3500 7725 3500
+	4925 2600 4700 2600
 Wire Wire Line
-	8550 4175 8550 3700
+	4700 2600 4700 4150
 Wire Wire Line
-	8550 3700 7725 3700
+	4700 4150 6025 4150
 Wire Wire Line
-	4925 4175 8550 4175
+	5525 2600 5750 2600
 Wire Wire Line
-	6350 3500 6550 3500
+	5750 2600 5750 4475
 Wire Wire Line
-	6425 2600 6425 3100
+	5750 4475 6025 4475
 Wire Wire Line
-	6425 3100 6550 3100
+	5225 2400 4850 2400
 Wire Wire Line
-	4325 2600 4325 3375
+	4850 2400 4850 4750
 Wire Wire Line
-	4325 3375 6550 3375
+	4850 4750 6025 4750
 Wire Wire Line
-	6550 3375 6550 3300
+	6325 4750 6850 4750
+Wire Wire Line
+	6850 4750 6850 3500
+Wire Wire Line
+	6325 4475 6750 4475
+Wire Wire Line
+	6750 4475 6750 3300
+Wire Wire Line
+	6750 3300 7125 3300
+Wire Wire Line
+	6325 4150 6625 4150
+Wire Wire Line
+	6625 4150 6625 3100
+Wire Wire Line
+	6625 3100 7125 3100
+Wire Wire Line
+	4925 2800 4925 5050
+Wire Wire Line
+	4925 5050 7850 5050
+Wire Wire Line
+	7850 5050 7850 3700
+Wire Wire Line
+	7850 3700 7725 3700
+Wire Wire Line
+	7725 3500 7900 3500
+Wire Wire Line
+	7900 3500 7900 5025
+Wire Wire Line
+	7900 5025 5525 5025
+Wire Wire Line
+	5525 5025 5525 2800
 $EndSCHEMATC

Commit message: V1.4 - the colour pins go to the right places now
Parts:
- R3: value 150 -> RBlue
- renumbered R2 to RGreen, R1 to RRed
Connections:
- wire segments 35 -> 37
Changed lines of the file:
@@
 EESchema Schematic File Version 4
+LIBS:PC8801mkII VGA-cache
 EELAYER 26 0
 EELAYER END
@@
 GND
 Text Label 4925 2600 2    50   ~ 0
+Green
+Text Label 5525 2600 0    50   ~ 0
 Red
-Text Label 5525 2600 0    50   ~ 0
-Green
 Text Label 5225 2400 0    50   ~ 0
 Blue
@@
 NoConn ~ 4925 2700
 $Comp
-L Device:R R1
+L Device:R RRed
 U 1 1 5B82F80D
 P 6175 4150
-F 0 "R1" V 5968 4150 50  0000 C CNN
+F 0 "RRed" V 5968 4150 50  0000 C CNN
 F 1 "150" V 6059 4150 50  0000 C CNN
 F 2 "Resistors_ThroughHole:R_Axial_DIN0204_L3.6mm_D1.6mm_P5.08mm_Horizontal" V 6105 4150 50  0001 C CNN
@@
 $EndComp
 $Comp
-L Device:R R2
+L Device:R RGreen
 U 1 1 5B82FD72
 P 6175 4475
-F 0 "R2" V 5968 4475 50  0000 C CNN
+F 0 "RGreen" V 5968 4475 50  0000 C CNN
 F 1 "150" V 6059 4475 50  0000 C CNN
 F 2 "Resistors_ThroughHole:R_Axial_DIN0204_L3.6mm_D1.6mm_P5.08mm_Horizontal" V 6105 4475 50  0001 C CNN
@@
 P 6175 4750
 F 0 "R3" V 5968 4750 50  0000 C CNN
-F 1 "150" V 6059 4750 50  0000 C CNN
+F 1 "RBlue" V 6059 4750 50  0000 C CNN
 F 2 "Resistors_ThroughHole:R_Axial_DIN0204_L3.6mm_D1.6mm_P5.08mm_Horizontal" V 6105 4750 50  0001 C CNN
 F 3 "~" H 6175 4750 50  0001 C CNN
@@
 $EndComp
 Wire Wire Line
-	4925 2600 4700 2600
-Wire Wire Line
-	4700 2600 4700 4150
-Wire Wire Line
 	4700 4150 6025 4150
-Wire Wire Line
-	5525 2600 5750 2600
-Wire Wire Line
-	5750 2600 5750 4475
-Wire Wire Line
-	5750 4475 6025 4475
 Wire Wire Line
 	5225 2400 4850 2400
@@
 Wire Wire Line
 	5525 5025 5525 2800
+Wire Wire Line
+	4275 4475 4275 2600
+Wire Wire Line
+	4275 2600 4925 2600
+Wire Wire Line
+	4275 4475 6025 4475
+Wire Wire Line
+	4700 4150 4700 3075
+Wire Wire Line
+	4700 3075 5775 3075
+Wire Wire Line
+	5775 3075 5775 2600
+Wire Wire Line
+	5525 2600 5775 2600
 $EndSCHEMATC

Commit message: Auto-bodge
Parts:
- renumbered RGreen to RGreen1, RRed to RRed1
Changed lines of the file:
@@
 NoConn ~ 4925 2700
 $Comp
-L Device:R RRed
+L Device:R RRed1
 U 1 1 5B82F80D
 P 6175 4150
-F 0 "RRed" V 5968 4150 50  0000 C CNN
+F 0 "RRed1" V 5968 4150 50  0000 C CNN
 F 1 "150" V 6059 4150 50  0000 C CNN
 F 2 "Resistors_ThroughHole:R_Axial_DIN0204_L3.6mm_D1.6mm_P5.08mm_Horizontal" V 6105 4150 50  0001 C CNN
@@
 $EndComp
 $Comp
-L Device:R RGreen
+L Device:R RGreen1
 U 1 1 5B82FD72
 P 6175 4475
-F 0 "RGreen" V 5968 4475 50  0000 C CNN
+F 0 "RGreen1" V 5968 4475 50  0000 C CNN
 F 1 "150" V 6059 4475 50  0000 C CNN
 F 2 "Resistors_ThroughHole:R_Axial_DIN0204_L3.6mm_D1.6mm_P5.08mm_Horizontal" V 6105 4475 50  0001 C CNN

Commit message: Add warning label telling people the port is backwards from how it comes out of the PC88
Other:
- note added: "Note: this is HORIZONTALLY FLIPPED from how the port is,\nlooking at the back of the computer.\n(e.g. looking at the back of the computer, Green is on the RIGHT)"
Changed lines of the file:
@@
 Wire Wire Line
 	5525 2600 5775 2600
+Text Notes 5600 2400 0    50   ~ 0
+Note: this is HORIZONTALLY FLIPPED from how the port is,\nlooking at the back of the computer.\n(e.g. looking at the back of the computer, Green is on the RIGHT)
 $EndSCHEMATC

Commit message: Bigger resistors, trying to shorten colour tracks, run sync far away from all colours
Parts:
- R3, RGreen1, RRed1: footprint Resistors_ThroughHole:R_Axial_DIN0204_L3.6mm_D1.6mm_P5.08mm_Horizontal -> Resistors_ThroughHole:R_Axial_DIN0204_L3.6mm_D1.6mm_P7.62mm_Horizontal
Changed lines of the file:
@@
 F 0 "RRed1" V 5968 4150 50  0000 C CNN
 F 1 "150" V 6059 4150 50  0000 C CNN
-F 2 "Resistors_ThroughHole:R_Axial_DIN0204_L3.6mm_D1.6mm_P5.08mm_Horizontal" V 6105 4150 50  0001 C CNN
+F 2 "Resistors_ThroughHole:R_Axial_DIN0204_L3.6mm_D1.6mm_P7.62mm_Horizontal" V 6105 4150 50  0001 C CNN
 F 3 "~" H 6175 4150 50  0001 C CNN
 	1    6175 4150
@@
 F 0 "RGreen1" V 5968 4475 50  0000 C CNN
 F 1 "150" V 6059 4475 50  0000 C CNN
-F 2 "Resistors_ThroughHole:R_Axial_DIN0204_L3.6mm_D1.6mm_P5.08mm_Horizontal" V 6105 4475 50  0001 C CNN
+F 2 "Resistors_ThroughHole:R_Axial_DIN0204_L3.6mm_D1.6mm_P7.62mm_Horizontal" V 6105 4475 50  0001 C CNN
 F 3 "~" H 6175 4475 50  0001 C CNN
 	1    6175 4475
@@
 F 0 "R3" V 5968 4750 50  0000 C CNN
 F 1 "RBlue" V 6059 4750 50  0000 C CNN
-F 2 "Resistors_ThroughHole:R_Axial_DIN0204_L3.6mm_D1.6mm_P5.08mm_Horizontal" V 6105 4750 50  0001 C CNN
+F 2 "Resistors_ThroughHole:R_Axial_DIN0204_L3.6mm_D1.6mm_P7.62mm_Horizontal" V 6105 4750 50  0001 C CNN
 F 3 "~" H 6175 4750 50  0001 C CNN
 	1    6175 4750
