File: PC8801mkII VGA.sch (KiCad schematic (older format))
At the start: 5 parts

Commit message: Flipping 12V and Bonus aroundg
Other:
- note added: "Note: this is HORIZONTALLY FLIPPED from how the port is,\nlooking at the back of the computer.\n(e.g. looking at the back of the computer, Green is on the RIGHT)\n\nThis means that pin numbers DO NOT line up with what you read on \nother schematics."
- note removed: "Note: this is HORIZONTALLY FLIPPED from how the port is,\nlooking at the back of the computer.\n(e.g. looking at the back of the computer, Green is on the RIGHT)"
Changed lines of the file:
@@
 EESchema Schematic File Version 4
 LIBS:PC8801mkII VGA-cache
-EELAYER 26 0
+EELAYER 30 0
 EELAYER END
 $Descr A4 11693 8268
@@
 Text Label 5225 2400 0    50   ~ 0
 Blue
-Text Label 4925 2700 2    50   ~ 0
-NC
 NoConn ~ 5525 2700
 Text Label 4925 2800 2    50   ~ 0
@@
 Wire Wire Line
 	6850 3500 7125 3500
-Text Label 5525 2700 0    50   ~ 0
-12V
 Wire Wire Line
 	5225 3400 5225 3800
@@
 	5525 2600 5775 2600
 Text Notes 5600 2400 0    50   ~ 0
-Note: this is HORIZONTALLY FLIPPED from how the port is,\nlooking at the back of the computer.\n(e.g. looking at the back of the computer, Green is on the RIGHT)
+Note: this is HORIZONTALLY FLIPPED from how the port is,\nlooking at the back of the computer.\n(e.g. looking at the back of the computer, Green is on the RIGHT)\n\nThis means that pin numbers DO NOT line up with what you read on \nother schematics.
+Text Label 4925 2700 2    50   ~ 0
+12V
+Text Label 5525 2700 0    50   ~ 0
+NC
 $EndSCHEMATC

Commit message: Wait - the pin numbers were right in the first place
Other:
- note added: "Note: this is HORIZONTALLY FLIPPED from how the port is,\nlooking at the back of the computer.\n(e.g. looking at the back of the computer, Green is on the RIGHT)"
- note removed: "Note: this is HORIZONTALLY FLIPPED from how the port is,\nlooking at the back of the computer.\n(e.g. looking at the back of the computer, Green is on the RIGHT)\n\nThis means that pin numbers DO NOT line up with what you read on \nother schematics."
Changed lines of the file:
@@
 	5525 2600 5775 2600
 Text Notes 5600 2400 0    50   ~ 0
-Note: this is HORIZONTALLY FLIPPED from how the port is,\nlooking at the back of the computer.\n(e.g. looking at the back of the computer, Green is on the RIGHT)\n\nThis means that pin numbers DO NOT line up with what you read on \nother schematics.
+Note: this is HORIZONTALLY FLIPPED from how the port is,\nlooking at the back of the computer.\n(e.g. looking at the back of the computer, Green is on the RIGHT)
 Text Label 4925 2700 2    50   ~ 0
+NC
+Text Label 5525 2700 0    50   ~ 0
 12V
-Text Label 5525 2700 0    50   ~ 0
-NC
 $EndSCHEMATC

Commit message: Fix the callout
Other:
- note added: "Looking at the back of the computer, green is on the left side"
- note removed: "Note: this is HORIZONTALLY FLIPPED from how the port is,\nlooking at the back of the computer.\n(e.g. looking at the back of the computer, Green is on the RIGHT)"
Changed lines of the file:
@@
 EESchema Schematic File Version 4
-LIBS:PC8801mkII VGA-cache
 EELAYER 30 0
 EELAYER END
@@
 	5525 2600 5775 2600
 Text Notes 5600 2400 0    50   ~ 0
-Note: this is HORIZONTALLY FLIPPED from how the port is,\nlooking at the back of the computer.\n(e.g. looking at the back of the computer, Green is on the RIGHT)
+Looking at the back of the computer, green is on the left side
 Text Label 4925 2700 2    50   ~ 0
 NC

Commit message: Move 12V to the right side
Connections:
- net labels removed: NC
Changed lines of the file:
@@
 Looking at the back of the computer, green is on the left side
 Text Label 4925 2700 2    50   ~ 0
-NC
-Text Label 5525 2700 0    50   ~ 0
 12V
 $EndSCHEMATC

Commit message: Cleaning up
Parts:
- RBlue1: renamed from R3; value RBlue -> 150Ω
- RGreen1, RRed1: value 150 -> 150Ω
Changed lines of the file:
@@
 P 6175 4150
 F 0 "RRed1" V 5968 4150 50  0000 C CNN
-F 1 "150" V 6059 4150 50  0000 C CNN
+F 1 "150Ω" V 6059 4150 50  0000 C CNN
 F 2 "Resistors_ThroughHole:R_Axial_DIN0204_L3.6mm_D1.6mm_P7.62mm_Horizontal" V 6105 4150 50  0001 C CNN
 F 3 "~" H 6175 4150 50  0001 C CNN
@@
 P 6175 4475
 F 0 "RGreen1" V 5968 4475 50  0000 C CNN
-F 1 "150" V 6059 4475 50  0000 C CNN
+F 1 "150Ω" V 6059 4475 50  0000 C CNN
 F 2 "Resistors_ThroughHole:R_Axial_DIN0204_L3.6mm_D1.6mm_P7.62mm_Horizontal" V 6105 4475 50  0001 C CNN
 F 3 "~" H 6175 4475 50  0001 C CNN
@@
 $EndComp
 $Comp
-L Device:R R3
+L Device:R RBlue1
 U 1 1 5B82FE62
-P 6175 4750
-F 0 "R3" V 5968 4750 50  0000 C CNN
-F 1 "RBlue" V 6059 4750 50  0000 C CNN
-F 2 "Resistors_ThroughHole:R_Axial_DIN0204_L3.6mm_D1.6mm_P7.62mm_Horizontal" V 6105 4750 50  0001 C CNN
-F 3 "~" H 6175 4750 50  0001 C CNN
-	1    6175 4750
+P 6175 4800
+F 0 "RBlue1" V 5968 4800 50  0000 C CNN
+F 1 "150Ω" V 6059 4800 50  0000 C CNN
+F 2 "Resistors_ThroughHole:R_Axial_DIN0204_L3.6mm_D1.6mm_P7.62mm_Horizontal" V 6105 4800 50  0001 C CNN
+F 3 "~" H 6175 4800 50  0001 C CNN
+	1    6175 4800
 	0    1    1    0
 $EndComp
@@
 	4850 2400 4850 4750
 Wire Wire Line
-	4850 4750 6025 4750
+	4850 4750 6025 4800
 Wire Wire Line
-	6325 4750 6850 4750
+	6325 4800 6850 4750
 Wire Wire Line
 	6850 4750 6850 3500

Commit message: Use decoupling caps
Parts:
- added C1, C2, C3: 0.1µF, Capacitor_SMD:C_0805_2012Metric_Pad1.15x1.40mm_HandSolder, symbol Device:C_Small
Connections:
- wire segments 37 -> 48
Changed lines of the file:
@@
 Wire Wire Line
 	6850 3500 7125 3500
-Wire Wire Line
-	5225 3400 5225 3800
 NoConn ~ 7125 3600
 Connection ~ 5225 3000
@@
 	6325 4800 6850 4750
 Wire Wire Line
-	6850 4750 6850 3500
-Wire Wire Line
 	6325 4475 6750 4475
-Wire Wire Line
-	6750 4475 6750 3300
 Wire Wire Line
 	6750 3300 7125 3300
@@
 	6325 4150 6625 4150
 Wire Wire Line
-	6625 4150 6625 3100
+	6625 4150 6625 3550
 Wire Wire Line
 	6625 3100 7125 3100
@@
 Text Label 4925 2700 2    50   ~ 0
 12V
+$Comp
+L Device:C_Small C3
+U 1 1 605A2EFB
+P 6525 3550
+F 0 "C3" V 6296 3550 50  0000 C CNN
+F 1 "0.1µF" V 6387 3550 50  0000 C CNN
+F 2 "Capacitor_SMD:C_0805_2012Metric_Pad1.15x1.40mm_HandSolder" H 6525 3550 50  0001 C CNN
+F 3 "~" H 6525 3550 50  0001 C CNN
+	1    6525 3550
+	0    1    1    0
+$EndComp
+Connection ~ 6625 3550
+Wire Wire Line
+	6625 3550 6625 3100
+Connection ~ 6850 3775
+Wire Wire Line
+	6850 3775 6850 4750
+$Comp
+L Device:C_Small C2
+U 1 1 605A51E3
+P 6200 3650
+F 0 "C2" V 5971 3650 50  0000 C CNN
+F 1 "0.1µF" V 6062 3650 50  0000 C CNN
+F 2 "Capacitor_SMD:C_0805_2012Metric_Pad1.15x1.40mm_HandSolder" H 6200 3650 50  0001 C CNN
+F 3 "~" H 6200 3650 50  0001 C CNN
+	1    6200 3650
+	0    1    1    0
+$EndComp
+Wire Wire Line
+	5800 3775 6850 3775
+$Comp
+L Device:C_Small C1
+U 1 1 605A6432
+P 5700 3775
+F 0 "C1" V 5471 3775 50  0000 C CNN
+F 1 "0.1µF" V 5562 3775 50  0000 C CNN
+F 2 "Capacitor_SMD:C_0805_2012Metric_Pad1.15x1.40mm_HandSolder" H 5700 3775 50  0001 C CNN
+F 3 "~" H 5700 3775 50  0001 C CNN
+	1    5700 3775
+	0    1    1    0
+$EndComp
+Wire Wire Line
+	6425 3550 5225 3550
+Wire Wire Line
+	5225 3400 5225 3550
+Connection ~ 5225 3550
+Wire Wire Line
+	5225 3550 5225 3650
+Wire Wire Line
+	6100 3650 5225 3650
+Connection ~ 5225 3650
+Wire Wire Line
+	5225 3650 5225 3775
+Wire Wire Line
+	5600 3775 5225 3775
+Connection ~ 5225 3775
+Wire Wire Line
+	5225 3775 5225 3800
+Wire Wire Line
+	6750 3300 6750 3650
+Wire Wire Line
+	6850 3500 6850 3775
+Wire Wire Line
+	6300 3650 6750 3650
+Connection ~ 6750 3650
+Wire Wire Line
+	6750 3650 6750 4475
 $EndSCHEMATC
