File: PC8801mkII VGA.kicad_sch (KiCad schematic)
At the start: 5 parts

Commit message: v1.9 test release
Parts:
- added C1, C2, C3: 0.1µF, Capacitor_THT:C_Disc_D3.4mm_W2.1mm_P2.50mm, symbol Device:C_Small
Connections:
- net Blue_VGA: now also C3.2; no longer R3.1
- net Green_VGA: now also C2.2; no longer R2.1
- net Red_VGA: now also C1.2; no longer R1.1
- new net: C3.1, R3.1
- new net: C2.1, R2.1
- new net: C1.1, R1.1
